File: soundboard.kicad_sch (KiCad schematic)
At the start: 0 parts

Commit message: finished KiCad
Parts:
- added C1: C, Capacitor_THT:C_Radial_D8.0mm_H11.5mm_P3.50mm, symbol Device:C
- added D1, D10, D11, D12, D13, D14, D15, D16, D2, D3, D4, D5, D6, D7, D8, D9: D, Diode_THT:D_DO-35_SOD27_P7.62mm_Horizontal, symbol Device:D
- added D17, D18, D19, D20, D21, D22, D23, D24, D25, D26, D27, D28, D29, D30, D31, D32: SK6812MINI, LED_SMD:LED_SK6812MINI_PLCC4_3.5x3.5mm_P1.75mm, symbol LED:SK6812MINI
- added J1: Conn_01x04, Connector_PinHeader_2.54mm:PinHeader_1x04_P2.54mm_Vertical, symbol Connector_Generic:Conn_01x04
- added SW1, SW10, SW11, SW12, SW13, SW14, SW15, SW16, SW2, SW3, SW4, SW5, SW6, SW7, SW8, SW9: SW_Push_45deg, Button_Switch_Keyboard:SW_Cherry_MX_1.00u_PCB, symbol Switch:SW_Push_45deg
- added U1: MOUDLE-SEEEDUINO-XIAO, footprints:XIAO-Generic-Hybrid-14P-2.54-21X17.8MM, symbol XIAO_RP2040:MOUDLE-SEEEDUINO-XIAO
Connections:
- new net: D7.2 (A), SW7.2
- new net: D27.1 (DOUT), D28.3 (DIN)
- new net: D26.1 (DOUT), D27.3 (DIN)
- new net: D22.1 (DOUT), D23.3 (DIN)
- new net: D21.1 (DOUT), D22.3 (DIN)
- new net: D31.1 (DOUT), D32.3 (DIN)
- new net: D5.2 (A), SW5.2
- new net: D11.2 (A), SW11.2
- new net: D10.2 (A), SW10.2
- new net: D14.2 (A), SW14.2
- new net: D28.1 (DOUT), D29.3 (DIN)
- new net: D9.2 (A), SW9.2
- new net: D13.2 (A), SW13.2
- new net: D12.2 (A), SW12.2
- new net: D17.1 (DOUT), D18.3 (DIN)
- new net: D2.2 (A), SW2.2
- new net: D30.1 (DOUT), D31.3 (DIN)
- new net: D20.1 (DOUT), D21.3 (DIN)
- new net: D19.1 (DOUT), D20.3 (DIN)
- new net: D8.2 (A), SW8.2
- new net: D1.2 (A), SW1.2
- new net: D4.2 (A), SW4.2
- new net: D16.2 (A), SW16.2
- new net: D23.1 (DOUT), D24.3 (DIN)
- new net: D29.1 (DOUT), D30.3 (DIN)
- new net: D24.1 (DOUT), D25.3 (DIN)
- new net: D15.2 (A), SW15.2
- new net: D6.2 (A), SW6.2
- new net: D18.1 (DOUT), D19.3 (DIN)
- new net: D3.2 (A), SW3.2
- new net: D25.1 (DOUT), D26.3 (DIN)
- new net +3V3: J1.2 (Pin_2), U1.12 (3V3)
- new net +5V: C1.1, D17.4 (VDD), D18.4 (VDD), D19.4 (VDD), D20.4 (VDD), D21.4 (VDD), D22.4 (VDD), D23.4 (VDD), D24.4 (VDD), D25.4 (VDD), D26.4 (VDD), D27.4 (VDD), D28.4 (VDD), D29.4 (VDD), D30.4 (VDD), D31.4 (VDD), D32.4 (VDD), U1.14 (5V)
- new net Column 0: SW1.1, SW13.1, SW5.1, SW9.1, U1.7 (PB08_A6_D6_TX)
- new net Column 1: SW10.1, SW14.1, SW2.1, SW6.1, U1.8 (PB09_A7_D7_RX)
- new net Column 2: SW11.1, SW15.1, SW3.1, SW7.1, U1.9 (PA7_A8_D8_SCK)
- new net Column 3: SW12.1, SW16.1, SW4.1, SW8.1, U1.10 (PA5_A9_D9_MISO)
- new net GND: C1.2, D17.2 (VSS), D18.2 (VSS), D19.2 (VSS), D20.2 (VSS), D21.2 (VSS), D22.2 (VSS), D23.2 (VSS), D24.2 (VSS), D25.2 (VSS), D26.2 (VSS), D27.2 (VSS), D28.2 (VSS), D29.2 (VSS), D30.2 (VSS), D31.2 (VSS), D32.2 (VSS), J1.1 (Pin_1), U1.13 (GND)
- new net LED: D17.3 (DIN), U1.11 (PA6_A10_D10_MOSI)
- new net OLED_SCL: J1.3 (Pin_3), U1.6 (PA9_A5_D5_SCL)
- new net OLED_SDA: J1.4 (Pin_4), U1.5 (PA8_A4_D4_SDA)
- new net Row 0: D1.1 (K), D2.1 (K), D3.1 (K), D4.1 (K), U1.1 (PA02_A0_D0)
- new net Row 1: D5.1 (K), D6.1 (K), D7.1 (K), D8.1 (K), U1.2 (PA4_A1_D1)
- new net Row 2: D10.1 (K), D11.1 (K), D12.1 (K), D9.1 (K), U1.3 (PA10_A2_D2)
- new net Row 3: D13.1 (K), D14.1 (K), D15.1 (K), D16.1 (K), U1.4 (PA11_A3_D3)
- no-connect marks 0 -> 1
