File: PCB/soundboard.kicad_pcb (KiCad board)
At the start: 2 copper layers, 82.2 x 103 mm, 51 parts, among them J1 Conn_01x04, SW1 SW_Push_45deg, SW10 SW_Push_45deg, SW11 SW_Push_45deg, SW12 SW_Push_45deg, SW13 SW_Push_45deg, SW14 SW_Push_45deg, SW15 SW_Push_45deg, SW16 SW_Push_45deg, SW2 SW_Push_45deg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

Commit message: update
Parts:
- removed C1: C, Capacitor_THT:C_Radial_D8.0mm_H11.5mm_P3.50mm
- added R1: R, Resistor_SMD:R_0805_2012Metric, B.Cu at (161.6, 55.6)
- D17, D18, D19, D20, D21, D22, D23, D24, D25, D26, D27, D28, D29, D30, D31, D32: footprint LED_SMD:LED_SK6812MINI_PLCC4_3.5x3.5mm_P1.75mm -> footprints:SK6812MINI-E_fixed
- moved D26 0.68 mm to (163.6, 121.5)
- moved D28 0.54 mm to (201.7, 121.5)
- moved D25 0.54 mm to (144.5, 121.5)
- moved D32 0.52 mm to (201.7, 140.5)
- moved D27 0.51 mm to (182.6, 121.5)
- moved D20 0.50 mm to (201.7, 83.4)
- moved D22 0.50 mm to (163.6, 102.4)
- moved D18 0.50 mm to (163.6, 83.4)
- moved D23 0.47 mm to (182.6, 102.4)
- moved D24 0.47 mm to (201.7, 102.4)
- moved D17 0.47 mm to (144.5, 83.4)
- moved D29 0.46 mm to (144.5, 140.5)
- moved D31 0.45 mm to (182.6, 140.5)
- moved D21 0.44 mm to (144.5, 102.4)
- moved D19 0.39 mm to (182.6, 83.4)
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Connections:
- U1 pad 11: LED -> Net-(U1-PA6_A10_D10_MOSI)
Routing:
- net +5V: track 460.1 -> 342.2 mm, vias 25 -> 4
- net GND: track 498.6 -> 423.1 mm, vias 20 -> 5
- net Net-(D24-DOUT): track 94.2 -> 77.1 mm
- net Row 3: track 163.1 -> 147.2 mm, vias 1 -> 0
- net Row 2: track 143.6 -> 131.2 mm
- net Net-(D20-DOUT): track 92.5 -> 81.4 mm, vias 0 -> 2
- net Net-(U1-PA6_A10_D10_MOSI): track 0.00 -> 9.32 mm
- net /OLED_SDA: track 82.3 -> 73.1 mm
- net Column 3: track 113.6 -> 122.5 mm
- net Column 2: track 93.5 -> 101.8 mm
- net Column 1: track 73.4 -> 78.8 mm
- net Net-(D28-DOUT): track 99.0 -> 103.9 mm
- net LED: track 42.0 -> 46.7 mm, vias 1 -> 3
- net Net-(D17-DOUT): track 16.3 -> 20.4 mm, vias 0 -> 2
- net Net-(D22-DOUT): track 16.3 -> 20.1 mm
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